Commit message: unfixed pid

File: urdf/omni_robot/camera.xacro (robot description, xacro)
@@ -24,5 +24,5 @@
         <parent link="base_link"/>
         <child link="camera_link"/>
-        <origin xyz="0 0 0" rpy="0 0 0"/>
+        <origin xyz="0 0 0.125" rpy="0 0 0"/>
     </joint>
     <!-- LiDAR 传感器（GPU LiDAR，装在 camera_link 上） -->

File: urdf/omni_robot/mobile_base.xacro (robot description, xacro)
@@ -24,4 +24,5 @@
                 <material name="${color}"/>
             </visual>
+            <!-- cylinder 碰撞在 DART+ODE 中与非轴对齐平面碰撞时 AABB 溢出，注释备用 -->
             <collision>
                 <geometry>
@@ -30,4 +31,10 @@
                 <origin xyz="0 0 0" rpy="${pi/2.0} 0 0"/>
             </collision>
+            <!-- <collision>
+                <geometry>
+                    <box size="${2*wheel_radius} 0.04 ${2*wheel_radius}"/>
+                </geometry>
+                <origin xyz="0 0 0" rpy="${pi/2.0} 0 0"/>
+            </collision> -->
             <xacro:cylinder_inertia m="${wheel_mass}" r="${wheel_radius}" l="${wheel_length}"
                                     o_xyz="0 0 0" o_rpy="${pi/2.0} 0 0"/>
@@ -35,5 +42,12 @@
     </xacro:macro>
     <!-- ========== 基座标系 ========== -->
-    <link name="base_footprint"/>
+    <!-- DART 要求所有参与运动链的 link 必须有质量/惯性，
+         否则 body node 位姿为 NaN → ODE 碰撞 AABB 溢出 -->
+    <link name="base_footprint">
+        <inertial>
+            <mass value="0.001"/>
+            <inertia ixx="1e-6" ixy="0" ixz="0" iyy="1e-6" iyz="0" izz="1e-6"/>
+        </inertial>
+    </link>
     <!-- ========== 底盘 link ========== -->
     <link name="base_link">

File: urdf/omni_robot/mobile_base_gazebo.xacro (robot description, xacro)
@@ -1,8 +1,5 @@
 <?xml version="1.0"?>
 <robot xmlns:xacro="https://www.ros.org/wiki/xacro">
-    <!-- ========== 全向轮摩擦 ========== -->
-    <!-- mu1: 高摩擦方向 (fdir1 = 轮子滚动方向 = 本地 X 轴) -->
-    <!-- mu2: 低摩擦方向 (垂直于 fdir1 = 本地 Y 轴 = 滚子自由滑动方向) -->
-    <!-- 滚子垂直于主轮：沿轮轴方向自由滑动 -->
+    <!-- ========== 全向轮摩擦（测试注释：排查 Ignition URDF→SDF 兼容性） ========== -->
     <gazebo reference="fl_wheel_link">
         <mu1>1.0</mu1>
@@ -52,4 +49,10 @@
             <wheel_separation_x>${omni_lx * 2}</wheel_separation_x>
             <wheel_separation_y>${omni_ly * 2}</wheel_separation_y>
+            <!-- PID 速度环参数：改这里无需重新编译 C++ -->
+            <pid_p>0.02</pid_p>
+            <pid_i>0.0</pid_i>
+            <pid_d>0.0005</pid_d>
+            <pid_cmd_max>0.5</pid_cmd_max>
+            <pid_cmd_min>-0.5</pid_cmd_min>
         </plugin>
     </gazebo>
